Commit message: Update spot.urdf.xacro

File: spot_description/urdf/spot.urdf.xacro (robot description, xacro)
@@ -4,10 +4,10 @@
         <visual>
             <geometry>
-                <mesh filename="package://spot_description/meshes/body.dae" />
-            </geometry>
-        </visual>
-        <collision>
-            <geometry>
-                <mesh filename="package://spot_description/meshes/body_collision.stl" />
+                <mesh filename="https://raw.githubusercontent.com/clearpathrobotics/spot_ros/master/spot_description/meshes/body.dae" />
+            </geometry>
+        </visual>
+        <collision>
+            <geometry>
+                <mesh filename="https://raw.githubusercontent.com/clearpathrobotics/spot_ros/master/spot_description/meshes/body_collision.stl" />
             </geometry>
         </collision>
@@ -34,10 +34,10 @@
         <visual>
             <geometry>
-                <mesh filename="package://spot_description/meshes/front_left_hip.dae" />
-            </geometry>
-        </visual>
-        <collision>
-            <geometry>
-                <mesh filename="package://spot_description/meshes/front_left_hip_collision.stl" />
+                <mesh filename="https://raw.githubusercontent.com/clearpathrobotics/spot_ros/master/spot_description/meshes/front_left_hip.dae" />
+            </geometry>
+        </visual>
+        <collision>
+            <geometry>
+                <mesh filename="https://raw.githubusercontent.com/clearpathrobotics/spot_ros/master/spot_description/meshes/front_left_hip_collision.stl" />
             </geometry>
         </collision>
@@ -53,10 +53,10 @@
         <visual>
             <geometry>
-                <mesh filename="package://spot_description/meshes/front_left_upper_leg.dae" />
-            </geometry>
-        </visual>
-        <collision>
-            <geometry>
-                <mesh filename="package://spot_description/meshes/front_left_upper_leg_collision.stl" />
+                <mesh filename="https://raw.githubusercontent.com/clearpathrobotics/spot_ros/master/spot_description/meshes/front_left_upper_leg.dae" />
+            </geometry>
+        </visual>
+        <collision>
+            <geometry>
+                <mesh filename="https://raw.githubusercontent.com/clearpathrobotics/spot_ros/master/spot_description/meshes/front_left_upper_leg_collision.stl" />
             </geometry>
         </collision>
@@ -72,10 +72,10 @@
         <visual>
             <geometry>
-                <mesh filename="package://spot_description/meshes/front_left_lower_leg.dae" />
-            </geometry>
-        </visual>
-        <collision>
-            <geometry>
-                <mesh filename="package://spot_description/meshes/front_left_lower_leg_collision.stl" />
+                <mesh filename="https://raw.githubusercontent.com/clearpathrobotics/spot_ros/master/spot_description/meshes/front_left_lower_leg.dae" />
+            </geometry>
+        </visual>
+        <collision>
+            <geometry>
+                <mesh filename="https://raw.githubusercontent.com/clearpathrobotics/spot_ros/master/spot_description/meshes/front_left_lower_leg_collision.stl" />
             </geometry>
         </collision>
@@ -91,10 +91,10 @@
         <visual>
             <geometry>
-                <mesh filename="package://spot_description/meshes/front_right_hip.dae" />
-            </geometry>
-        </visual>
-        <collision>
-            <geometry>
-                <mesh filename="package://spot_description/meshes/front_right_hip_collision.stl" />
+                <mesh filename="https://raw.githubusercontent.com/clearpathrobotics/spot_ros/master/spot_description/meshes/front_right_hip.dae" />
+            </geometry>
+        </visual>
+        <collision>
+            <geometry>
+                <mesh filename="https://raw.githubusercontent.com/clearpathrobotics/spot_ros/master/spot_description/meshes/front_right_hip_collision.stl" />
             </geometry>
         </collision>
@@ -110,10 +110,10 @@
         <visual>
             <geometry>
-                <mesh filename="package://spot_description/meshes/front_right_upper_leg.dae" />
-            </geometry>
-        </visual>
-        <collision>
-            <geometry>
-                <mesh filename="package://spot_description/meshes/front_right_upper_leg_collision.stl" />
+                <mesh filename="https://raw.githubusercontent.com/clearpathrobotics/spot_ros/master/spot_description/meshes/front_right_upper_leg.dae" />
+            </geometry>
+        </visual>
+        <collision>
+            <geometry>
+                <mesh filename="https://raw.githubusercontent.com/clearpathrobotics/spot_ros/master/spot_description/meshes/front_right_upper_leg_collision.stl" />
             </geometry>
         </collision>
@@ -129,10 +129,10 @@
         <visual>
             <geometry>
-                <mesh filename="package://spot_description/meshes/front_right_lower_leg.dae" />
-            </geometry>
-        </visual>
-        <collision>
-            <geometry>
-                <mesh filename="package://spot_description/meshes/front_right_lower_leg_collision.stl" />
+                <mesh filename="https://raw.githubusercontent.com/clearpathrobotics/spot_ros/master/spot_description/meshes/front_right_lower_leg.dae" />
+            </geometry>
+        </visual>
+        <collision>
+            <geometry>
+                <mesh filename="https://raw.githubusercontent.com/clearpathrobotics/spot_ros/master/spot_description/meshes/front_right_lower_leg_collision.stl" />
             </geometry>
         </collision>
@@ -148,10 +148,10 @@
         <visual>
             <geometry>
-                <mesh filename="package://spot_description/meshes/rear_left_hip.dae" />
-            </geometry>
-        </visual>
-        <collision>
-            <geometry>
-                <mesh filename="package://spot_description/meshes/rear_left_hip_collision.stl" />
+                <mesh filename="https://raw.githubusercontent.com/clearpathrobotics/spot_ros/master/spot_description/meshes/rear_left_hip.dae" />
+            </geometry>
+        </visual>
+        <collision>
+            <geometry>
+                <mesh filename="https://raw.githubusercontent.com/clearpathrobotics/spot_ros/master/spot_description/meshes/rear_left_hip_collision.stl" />
             </geometry>
         </collision>
@@ -167,10 +167,10 @@
         <visual>
             <geometry>
-                <mesh filename="package://spot_description/meshes/rear_left_upper_leg.dae" />
-            </geometry>
-        </visual>
-        <collision>
-            <geometry>
-                <mesh filename="package://spot_description/meshes/rear_left_upper_leg_collision.stl" />
+                <mesh filename="https://raw.githubusercontent.com/clearpathrobotics/spot_ros/master/spot_description/meshes/rear_left_upper_leg.dae" />
+            </geometry>
+        </visual>
+        <collision>
+            <geometry>
+                <mesh filename="https://raw.githubusercontent.com/clearpathrobotics/spot_ros/master/spot_description/meshes/rear_left_upper_leg_collision.stl" />
             </geometry>
         </collision>
@@ -186,10 +186,10 @@
         <visual>
             <geometry>
-                <mesh filename="package://spot_description/meshes/rear_left_lower_leg.dae" />
-            </geometry>
-        </visual>
-        <collision>
-            <geometry>
-                <mesh filename="package://spot_description/meshes/rear_left_lower_leg_collision.stl" />
+                <mesh filename="https://raw.githubusercontent.com/clearpathrobotics/spot_ros/master/spot_description/meshes/rear_left_lower_leg.dae" />
+            </geometry>
+        </visual>
+        <collision>
+            <geometry>
+                <mesh filename="https://raw.githubusercontent.com/clearpathrobotics/spot_ros/master/spot_description/meshes/rear_left_lower_leg_collision.stl" />
             </geometry>
         </collision>
@@ -205,10 +205,10 @@
         <visual>
             <geometry>
-                <mesh filename="package://spot_description/meshes/rear_right_hip.dae" />
-            </geometry>
-        </visual>
-        <collision>
-            <geometry>
-                <mesh filename="package://spot_description/meshes/rear_right_hip_collision.stl" />
+                <mesh filename="https://raw.githubusercontent.com/clearpathrobotics/spot_ros/master/spot_description/meshes/rear_right_hip.dae" />
+            </geometry>
+        </visual>
+        <collision>
+            <geometry>
+                <mesh filename="https://raw.githubusercontent.com/clearpathrobotics/spot_ros/master/spot_description/meshes/rear_right_hip_collision.stl" />
             </geometry>
         </collision>
@@ -224,10 +224,10 @@
         <visual>
             <geometry>
-                <mesh filename="package://spot_description/meshes/rear_right_upper_leg.dae" />
-            </geometry>
-        </visual>
-        <collision>
-            <geometry>
-                <mesh filename="package://spot_description/meshes/rear_right_upper_leg_collision.stl" />
+                <mesh filename="https://raw.githubusercontent.com/clearpathrobotics/spot_ros/master/spot_description/meshes/rear_right_upper_leg.dae" />
+            </geometry>
+        </visual>
+        <collision>
+            <geometry>
+                <mesh filename="https://raw.githubusercontent.com/clearpathrobotics/spot_ros/master/spot_description/meshes/rear_right_upper_leg_collision.stl" />
             </geometry>
         </collision>
@@ -243,10 +243,10 @@
         <visual>
             <geometry>
-                <mesh filename="package://spot_description/meshes/rear_right_lower_leg.dae" />
-            </geometry>
-        </visual>
-        <collision>
-            <geometry>
-                <mesh filename="package://spot_description/meshes/rear_right_lower_leg_collision.stl" />
+                <mesh filename="https://raw.githubusercontent.com/clearpathrobotics/spot_ros/master/spot_description/meshes/rear_right_lower_leg.dae" />
+            </geometry>
+        </visual>
+        <collision>
+            <geometry>
+                <mesh filename="https://raw.githubusercontent.com/clearpathrobotics/spot_ros/master/spot_description/meshes/rear_right_lower_leg_collision.stl" />
             </geometry>
         </collision>
@@ -259,7 +259,3 @@
         <limit effort="1000" velocity="1000.00" lower="-2.7929" upper="-0.257725" />
     </joint>
-    <!-- Standard accessories. -->
-    <xacro:include filename="$(find spot_description)/urdf/accessories.urdf.xacro" />
-    <!-- Optional custom includes. -->
-    <xacro:include filename="$(optenv SPOT_URDF_EXTRAS empty.urdf)" />
 </robot>

Commit message: Update spot.urdf.xacro

File: spot_description/urdf/spot.urdf.xacro (robot description, xacro)
@@ -43,5 +43,5 @@
         </collision>
     </link>
-    <joint name="front_left_hip_x" type="revolute">
+    <joint name="front_left_hip_x" type="floating">
         <origin xyz="0.29785 0.05500 0.00000" rpy="0 0 0" />
         <axis xyz="1 0 0" />
@@ -62,5 +62,5 @@
         </collision>
     </link>
-    <joint name="front_left_hip_y" type="revolute">
+    <joint name="front_left_hip_y" type="floating">
         <origin xyz="0.0 0.110945 0.0" rpy="0 0 0" />
         <axis xyz="0 1 0" />
@@ -81,5 +81,5 @@
         </collision>
     </link>
-    <joint name="front_left_knee" type="revolute">
+    <joint name="front_left_knee" type="floating">
         <origin xyz="0.025 0.000 -0.3205" rpy="0 0 0" />
         <axis xyz="0 1 0" />
@@ -100,5 +100,5 @@
         </collision>
     </link>
-    <joint name="front_right_hip_x" type="revolute">
+    <joint name="front_right_hip_x" type="floating">
         <origin xyz="0.29785 -0.05500 0.00000" rpy="0 0 0" />
         <axis xyz="1 0 0" />
@@ -119,5 +119,5 @@
         </collision>
     </link>
-    <joint name="front_right_hip_y" type="revolute">
+    <joint name="front_right_hip_y" type="floating">
         <origin xyz="0.0 -0.110945 0.0" rpy="0 0 0" />
         <axis xyz="0 1 0" />
@@ -138,5 +138,5 @@
         </collision>
     </link>
-    <joint name="front_right_knee" type="revolute">
+    <joint name="front_right_knee" type="floating">
         <origin xyz="0.025 0.000 -0.3205" rpy="0 0 0" />
         <axis xyz="0 1 0" />
@@ -157,5 +157,5 @@
         </collision>
     </link>
-    <joint name="rear_left_hip_x" type="revolute">
+    <joint name="rear_left_hip_x" type="floating">
         <origin xyz="-0.29785 0.05500 0.00000" rpy="0 0 0" />
         <axis xyz="1 0 0" />
@@ -176,5 +176,5 @@
         </collision>
     </link>
-    <joint name="rear_left_hip_y" type="revolute">
+    <joint name="rear_left_hip_y" type="floating">
         <origin xyz="0.0 0.110945 0.0" rpy="0 0 0" />
         <axis xyz="0 1 0" />
@@ -195,5 +195,5 @@
         </collision>
     </link>
-    <joint name="rear_left_knee" type="revolute">
+    <joint name="rear_left_knee" type="floating">
         <origin xyz="0.025 0.000 -0.3205" rpy="0 0 0" />
         <axis xyz="0 1 0" />
@@ -214,5 +214,5 @@
         </collision>
     </link>
-    <joint name="rear_right_hip_x" type="revolute">
+    <joint name="rear_right_hip_x" type="floating">
         <origin xyz="-0.29785 -0.05500 0.00000" rpy="0 0 0" />
         <axis xyz="1 0 0" />
@@ -233,5 +233,5 @@
         </collision>
     </link>
-    <joint name="rear_right_hip_y" type="revolute">
+    <joint name="rear_right_hip_y" type="floating">
         <origin xyz="0.0 -0.110945 0.0" rpy="0 0 0" />
         <axis xyz="0 1 0" />
@@ -252,5 +252,5 @@
         </collision>
     </link>
-    <joint name="rear_right_knee" type="revolute">
+    <joint name="rear_right_knee" type="floating">
         <origin xyz="0.025 0.000 -0.3205" rpy="0 0 0" />
         <axis xyz="0 1 0" />

Commit message: Update spot.urdf.xacro

File: spot_description/urdf/spot.urdf.xacro (robot description, xacro)
@@ -15,5 +15,5 @@
     <link name="base_link"/>
     <joint name="base_link_joint" type="fixed">
-        <origin xyz="0 0 0" rpy="0 0 0" />
+        <origin xyz="10 0 0" rpy="0 0 0" />
         <parent link="body" />
         <child link="base_link" />
